File: Radianite-Micro-F1C200s.kicad_sch (KiCad schematic)
At the start: 60 parts, among them J1 USB_C_Receptacle_USB2.0, J2 USB_B_Micro, J3 AudioJack4, J4 Conn_01x04, J5 Micro_SD_Card_Det2, J6 Conn_02x14_Counter_Clockwise, SW1 SW_Push, U1 F1C200s, U2 CH340E, U3 JW5211, U4 JW5211, U5 JW5211, U6 W25Q256JWPIQ, Y1 24MHz

Commit message: 2.9 change on micro
Connections:
- net +1V1: now also J6.24 (Pin_24)
- net +2V5: now also J6.25 (Pin_25)
- net D10: now reaches J6.21 (Pin_21)
- net D10: now also U1.16 (PD10/LCD_D14/DA_IN/EINTD10)
- net D9: now reaches J6.22 (Pin_22)
- net D9: now also U1.15 (PD9/LCD_D13/DA_LRCK/EINTD9)
- no-connect marks 44 -> 38
Changed lines of the file:
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@@
   (no_connect (at 143.51 114.3))
   (no_connect (at 143.51 182.88))
-  (no_connect (at 143.51 139.7))
+  (no_connect (at 143.51 134.62))
   (no_connect (at 71.12 101.6))
   (no_connect (at 39.37 106.68))
   (no_connect (at 252.73 185.42))
-  (no_connect (at 314.96 190.5))
   (no_connect (at 227.33 261.62))
   (no_connect (at 252.73 160.02))
   (no_connect (at 252.73 129.54))
-  (no_connect (at 314.96 198.12))
-  (no_connect (at 143.51 132.08))
   (no_connect (at 252.73 111.76))
   (no_connect (at 252.73 116.84))
   (no_connect (at 143.51 177.8))
-  (no_connect (at 143.51 134.62))
   (no_connect (at 50.8 59.69))
   (no_connect (at 143.51 157.48))
@@
   (no_connect (at 252.73 132.08))
   (no_connect (at 252.73 177.8))
-  (no_connect (at 314.96 195.58))
   (no_connect (at 143.51 162.56))
   (no_connect (at 252.73 187.96))
-  (no_connect (at 143.51 137.16))
   (no_connect (at 252.73 127))
-  (no_connect (at 314.96 187.96))
+  (no_connect (at 143.51 132.08))
   (no_connect (at 252.73 180.34))
   (no_connect (at 252.73 119.38))
@@
     (stroke (width 0) (type default))
   )
+  (wire (pts (xy 314.96 187.96) (xy 323.85 187.96))
+    (stroke (width 0) (type default))
+  )
   (wire (pts (xy 130.81 109.22) (xy 143.51 109.22))
     (stroke (width 0) (type default))
@@
     (stroke (width 0) (type default))
   )
+  (wire (pts (xy 314.96 190.5) (xy 327.66 190.5))
+    (stroke (width 0) (type default))
+  )
   (wire (pts (xy 320.04 200.66) (xy 314.96 200.66))
     (stroke (width 0) (type default))
@@
     (stroke (width 0) (type default))
   )
+  (wire (pts (xy 130.81 137.16) (xy 143.51 137.16))
+    (stroke (width 0) (type default))
+  )
   (wire (pts (xy 50.8 172.72) (xy 48.26 172.72))
     (stroke (width 0) (type default))
@@
     (stroke (width 0) (type default))
   )
+  (wire (pts (xy 314.96 198.12) (xy 321.31 198.12))
+    (stroke (width 0) (type default))
+  )
   (wire (pts (xy 314.96 213.36) (xy 321.31 213.36))
     (stroke (width 0) (type default))
@@
     (stroke (width 0) (type default))
   )
+  (wire (pts (xy 314.96 195.58) (xy 321.31 195.58))
+    (stroke (width 0) (type default))
+  )
+  (wire (pts (xy 130.81 139.7) (xy 143.51 139.7))
+    (stroke (width 0) (type default))
+  )
   (wire (pts (xy 323.85 48.26) (xy 323.85 50.8))
     (stroke (width 0) (type default))
@@
     (effects (font (size 1.27 1.27)) (justify left bottom))
   )
+  (label "D9" (at 130.81 137.16 0) (fields_autoplaced)
+    (effects (font (size 1.27 1.27)) (justify left bottom))
+  )
   (label "SOC_TX" (at 257.81 104.14 0) (fields_autoplaced)
     (effects (font (size 1.27 1.27)) (justify left bottom))
   )
+  (label "D10" (at 321.31 198.12 0) (fields_autoplaced)
+    (effects (font (size 1.27 1.27)) (justify left bottom))
+  )
   (label "D15" (at 130.81 152.4 0) (fields_autoplaced)
     (effects (font (size 1.27 1.27)) (justify left bottom))
@@
     (effects (font (size 1.27 1.27)) (justify left bottom))
   )
+  (label "D10" (at 130.81 139.7 0) (fields_autoplaced)
+    (effects (font (size 1.27 1.27)) (justify left bottom))
+  )
   (label "TF_DAT3" (at 189.23 243.84 0) (fields_autoplaced)
     (effects (font (size 1.27 1.27)) (justify left bottom))
@@
     (effects (font (size 1.27 1.27)) (justify left bottom))
   )
+  (label "D9" (at 321.31 195.58 0) (fields_autoplaced)
+    (effects (font (size 1.27 1.27)) (justify left bottom))
+  )
   (label "AV_R" (at 257.81 172.72 0) (fields_autoplaced)
     (effects (font (size 1.27 1.27)) (justify left bottom))
@@
     )
   )
+  (symbol (lib_id "power:+1V1") (at 327.66 190.5 0) (unit 1)
+    (in_bom yes) (on_board yes) (dnp no) (fields_autoplaced)
+    (property "Reference" "#PWR046" (at 327.66 194.31 0)
+      (effects (font (size 1.27 1.27)) hide)
+    )
+    (property "Value" "+1V1" (at 327.66 185.42 0)
+      (effects (font (size 1.27 1.27)))
+    )
+    (property "Footprint" "" (at 327.66 190.5 0)
+      (effects (font (size 1.27 1.27)) hide)
+    )
+    (property "Datasheet" "" (at 327.66 190.5 0)
+      (effects (font (size 1.27 1.27)) hide)
+    )
+    (pin "1")
+    (instances
+      (project "Radianite-Micro-F1C200s"
+        (path "/24fb9921-1e22-4a3d-9b11-ad2a65f2f75a"
+          (reference "#PWR046") (unit 1)
+        )
+      )
+    )
+  )
   (symbol (lib_id "Device:C") (at 330.2 55.88 90) (unit 1)
     (in_bom yes) (on_board yes) (dnp no)
@@
         )
       )
+    )
+  )
+  (symbol (lib_id "power:+2V5") (at 323.85 187.96 0) (unit 1)
+    (in_bom yes) (on_board yes) (dnp no) (fields_autoplaced)
+    (property "Reference" "#PWR045" (at 323.85 191.77 0)
+      (effects (font (size 1.27 1.27)) hide)
+    )
+    (property "Value" "+2V5" (at 323.85 182.88 0)
+      (effects (font (size 1.27 1.27)))
+    )
+    (property "Footprint" "" (at 323.85 187.96 0)
+      (effects (font (size 1.27 1.27)) hide)
+    )
+    (property "Datasheet" "" (at 323.85 187.96 0)
+      (effects (font (size 1.27 1.27)) hide)
+    )
+    (pin "1")
+    (instances
+      (project "Radianite-Micro-F1C200s"
+        (path "/24fb9921-1e22-4a3d-9b11-ad2a65f2f75a"
+          (reference "#PWR045") (unit 1)
+        )
+      )
