File: Radianite-Micro-F1C200s.kicad_pcb (KiCad board)
At the start: 2 copper layers, 60 x 28 mm, 73 parts, among them J1 USB_C_Receptacle_USB2.0, J2 USB_B_Micro, J3 AudioJack4, J4 Conn_01x04, J5 Micro_SD_Card_Det2, J6 Conn_02x14_Counter_Clockwise, SW1 SW_Push, U1 F1C200s, U2 CH340E, U3 JW5211, U4 JW5211, U5 JW5211, U6 W25Q256JWPIQ, Y1 24MHz

Commit message: minor drawing revision
Parts:
- moved J5 0.55 mm to (141.4, 121.7)
Routing:
- net Net-(D1-A): track 37.6 -> 77.8 mm
- net /RESET: track 33.0 -> 67.1 mm
- net /AV_R: track 49.8 -> 33.2 mm
- net /AV_L: track 27.2 -> 42.4 mm
- net /TF_DAT1: track 32.0 -> 45.1 mm
- net Net-(J4-Pin_2): track 10.9 -> 20.2 mm
- net /TF_DAT2: track 30.2 -> 37.6 mm
- net VBUS: track 76.6 -> 83.9 mm
- net +2V5: track 71.1 -> 77.8 mm
- net /SOC_TX: track 19.6 -> 25.2 mm
- net /FLASH_MISO: track 30.9 -> 35.9 mm
- net +1V1: track 49.5 -> 53.8 mm
- net /FLASH_SCK: track 47.4 -> 51.3 mm
- net +3V3: track 22.5 -> 25.9 mm
- net /SOC_DP: track 36.6 -> 39.9 mm
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Other:
- board text added: "* zeankun.dev didn't drew the israeli star"
- board text added: "Radianite Micro F1C200s"
