File: Radianite-Micro-F1C200s.kicad_pcb (KiCad board)
At the start: 2 copper layers, 60 x 28 mm, 73 parts, among them J1 USB_C_Receptacle_USB2.0, J2 USB_B_Micro, J3 AudioJack4, J4 Conn_01x04, J5 Micro_SD_Card_Det2, J6 Conn_02x14_Counter_Clockwise, SW1 SW_Push, U1 F1C200s, U2 CH340E, U3 JW5211, U4 JW5211, U5 JW5211, U6 W25Q256JWPIQ, Y1 24MHz

Commit message: declare v2.95
Routing:
- net /AV_VIDEO: track 62.8 -> 59.7 mm
- net /D6: track 24.2 -> 21.5 mm
- net /FLASH_SCK: track 51.3 -> 49.4 mm
- net +2V5: track 77.8 -> 78.8 mm
- net Net-(D1-A): track 77.8 -> 76.9 mm
- net /FLASH_CS: track 29.5 -> 28.8 mm
- net /D3: track 21.6 -> 22.2 mm
- net /D4: track 21.8 -> 22.5 mm
- net /D5: track 19.8 -> 20.5 mm
- net /TF_DAT1: track 45.1 -> 45.6 mm
Other:
- board text added: "r2.95"
- board text removed: "r2.9"
